File: PCB/RevExpansionHub.kicad_sch (KiCad schematic)
At the start: 3 parts, among them J14 Conn_01x03_Male

Commit message: added servo section
Parts:
- added C1, C2, C3, C4, C5, C59, C68, C76: 1uF, symbol Device:C
- added C5, C8: ?uF, symbol Device:C
- added C6: 22uF, symbol Device:C
- added D1, D2: SP0504BAHT, Package_TO_SOT_SMD:SOT-23-5, symbol Power_Protection:SP0504BAHT
- added F8: Polyfuse b2, symbol Device:Polyfuse_Small
- added J15: JTAG Connector, symbol Connector_Generic:Conn_01x06
- added J20: Servo Connector, symbol Connector_Generic:Conn_01x32
- added J5: Digital 6,7, symbol Connector:Conn_01x04_Pin
- added J6: Digital 4,5, symbol Connector:Conn_01x04_Pin
- added J7: Digital 2,3, symbol Connector:Conn_01x04_Pin
- added J8: Digital 0,1, symbol Connector:Conn_01x04_Pin
- added Q1, Q2, Q3, Q4, Q5, Q6, Q7, Q8: Q_NPN_EBC, symbol Device:Q_NPN_EBC
- added Q10, Q11, Q12, Q13, Q24, Q26, Q28, Q9: N32, symbol Device:Q_NPN_EBC
- added R1, R106, R113, R12, R121, R6, R9, R92: 33, symbol Device:R_Small
- added R10, R107, R114, R122, R13, R2, R4, R7: 44k, symbol Device:R_Small
- added R11, R110, R117, R125, R14, R3, R5, R8: 1000, symbol Device:R_Small
- added R16, R17, R18, R19, R20, R21, R22, R23, R24, R25, R26, R27, R28, R29, R30, R31, R32, R33, R34, R35, R36, R37, R38, R39: R_Small, symbol Device:R_Small
- added R44: 10k, symbol Device:R_Small
- gave numbers to parts that had none: 1
Connections:
- net GND: now also C1.2, C2.2, C3.2, C4.2, C5.2, C5.2, C59.2, C6.2, C68.2, C76.2, C8.2, J15.6 (Pin_6), J20.1 (Pin_1), J20.13 (Pin_13), J20.17 (Pin_17), J20.21 (Pin_21), J20.26 (Pin_26), J20.30 (Pin_30), J20.5 (Pin_5), J20.9 (Pin_9), J5.4 (Pin_4), J6.4 (Pin_4), J7.4 (Pin_4), J8.4 (Pin_4), Q1.1 (E), Q10.1 (E), Q11.1 (E), Q12.1 (E), Q13.1 (E), Q2.1 (E), Q24.1 (E), Q26.1 (E), Q28.1 (E), Q3.1 (E), Q4.1 (E), Q5.1 (E), Q6.1 (E), Q7.1 (E), Q8.1 (E), Q9.1 (E), R10.2, R107.2, R114.2, R122.2, R13.2, R2.2, R4.2, R7.2
- net at U11.1 (RO), U?.36 (PC4/U1RX): now also R44.2
- net at U11.8 (VCC): now also C5.1, C8.1
- net at U?.104 (PL4): now also R29.1
- net at U?.105 (PL3): now also R31.1
- net at U?.106 (PL2): now also R33.1
- net at U?.107 (PL1): now also R37.1
- net at U?.108 (PL0): now also R39.1
- net at U?.11 (PP2): now also Q7.2 (B), R24.2
- net TDO/SWO: now reaches U?.115 (PC3)
- net TDO/SWO: now also J15.5 (Pin_5)
- net TDI: now reaches U?.116 (PC2)
- net TDI: now also J15.4 (Pin_4)
- net TMS/SWDIO: now reaches U?.117 (PC1)
- net TMS/SWDIO: now also J15.3 (Pin_3)
- net SWCLK: now reaches U?.118 (PC0)
- net SWCLK: now also J15.2 (Pin_2)
- net at U?.127 (PJ4): now also Q6.2 (B), R30.2
- net at U?.128 (PJ5): now also Q5.2 (B), R28.2
- net at U?.21 (PH7): now also Q8.2 (B), R26.2
- net at U?.52 (PG3): now also R113.1
- net at U?.53 (PG2): now also R121.1
- net at U?.68 (PN7): now also Q3.2 (B), R32.2
- net at U?.69 (PN6): now also Q4.2 (B), R34.2
- net at U?.70 (PN5): now also Q2.2 (B), R36.2
- net at U?.71 (PN4): now also Q1.2 (B), R38.2
- net at U?.87 (PM2): now also R25.1
- net at U?.88 (PM1): now also R27.1
- new net: J8.1 (Pin_1), Q1.3 (C), R23.2, R39.2
- new net: Q11.2 (B), R6.2, R7.1
- new net: J6.2 (Pin_2), Q5.3 (C), R18.2, R29.2
- new net: Q10.2 (B), R4.1, R92.2
- new net: J7.1 (Pin_1), Q4.3 (C), R21.2, R35.2
- new net: J5.1 (Pin_1), Q8.3 (C), R17.2, R27.2
- new net: J5.2 (Pin_2), Q7.3 (C), R16.2, R25.2
- new net: J6.1 (Pin_1), Q6.3 (C), R19.2, R31.2
- new net: J7.2 (Pin_2), Q3.3 (C), R20.2, R33.2
- new net: Q13.3 (C), R14.2
- new net: Q9.3 (C), R3.2
- new net: J20.10 (Pin_10), J20.14 (Pin_14)
- new net: J20.18 (Pin_18), J20.22 (Pin_22)
- new net: Q9.2 (B), R1.2, R2.1
- new net: J8.2 (Pin_2), Q2.3 (C), R22.2, R37.2
- new net: Q24.2 (B), R106.2, R107.1
- new net: Q26.2 (B), R113.2, R114.1
- new net: Q12.2 (B), R10.1, R9.2
- new net: Q24.3 (C), R110.2
- new net: Q11.3 (C), R8.2
- new net: Q10.3 (C), R5.2
- new net: Q28.2 (B), R121.2, R122.1
- new net: Q13.2 (B), R12.2, R13.1
- new net: Q12.3 (C), R11.2
- new net +3.3V: J5.3 (Pin_3), J6.3 (Pin_3), J7.3 (Pin_3), J8.3 (Pin_3), R16.1, R17.1, R18.1, R19.1, R20.1, R21.1, R22.1, R23.1, R24.1, R26.1, R28.1, R30.1, R32.1, R34.1, R36.1, R38.1, R44.1
- new net +5V: C1.1, C2.1, C3.1, C4.1, C5.1, C59.1, C6.1, F8.1, J20.27 (Pin_27), J20.31 (Pin_31), R11.1, R110.1, R14.1, R3.1, R5.1, R8.1
- new net Fused_+5v_1: C68.1, C76.1, F8.2, J20.2 (Pin_2), J20.6 (Pin_6), R117.1, R125.1
- new net Servo0: J20.3 (Pin_3), Q28.3 (C), R125.2
- new net Servo1: J20.7 (Pin_7), Q26.3 (C), R117.2
- new net VDD: J15.1 (Pin_1)
- no-connect marks 0 -> 8
Other:
- note added: "Servo0"
- note added: "Servo1"
- note added: "Servo2"
- note added: "Servo3"
- note added: "Servo4"
- note added: "Servo5"
- moved on the sheet: J14, U11
