File: PCB/RevExpansionHub.kicad_sch (KiCad schematic)
At the start: 88 parts, among them J14 Conn_01x03_Male, J15 JTAG Connector, J20 Servo Connector, J5 Digital 6,7, J6 Digital 4,5, J7 Digital 2,3, J8 Digital 0,1, Q1 Q_NPN_EBC, Q10 N32, Q11 N32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

Commit message: Worked RS485 and serial
Parts:
- removed J14: Conn_01x03_Male, symbol Connector:Conn_01x03_Male
- added J1, J2, J3, J4: I2C, symbol Connector_Generic:Conn_01x04
- added J10, J16, J17, J9: Conn_01x04, symbol Connector_Generic:Conn_01x04
- added J11, J12: UART, symbol Connector_Generic:Conn_01x03
- added J13, J14: RS485, symbol Connector_Generic:Conn_01x03
- added R10, R4, R5, R6, R7 (x2), R8, R9: 2.49k, symbol Device:R_US
- added U9: SP0504BAHT, Package_TO_SOT_SMD:SOT-23-5, symbol Power_Protection:SP0504BAHT
Connections:
- net +3.3V: now also R10.1, R4.1, R5.1, R6.1, R7.1, R7.1, R8.1, R9.1
- net GND: now also J1.4 (Pin_4), J11.3 (Pin_3), J12.3 (Pin_3), J14.3 (Pin_3), J2.4 (Pin_4), J3.4 (Pin_4), J4.4 (Pin_4), U9.2 (A)
- net at U11.6 (A): now also J13.1 (Pin_1), J14.1 (Pin_1)
- net at U11.7 (B): now also J13.2 (Pin_2), J14.2 (Pin_2)
- net at U?.120 (PJ0): now also J12.2 (Pin_2), U9.4 (K)
- net at U?.121 (PJ1): now also J12.1 (Pin_1), U9.5 (K)
- net at U?.135 (PB5): now also J4.1 (Pin_1), R10.2
- net at U?.136 (PB4): now also J4.2 (Pin_2), R9.2
- net at U?.143 (PD6): now also J11.2 (Pin_2), U9.1 (K)
- net at U?.144 (PD7): now also J11.1 (Pin_1), U9.3 (K)
- new net: J3.1 (Pin_1), R8.2
- new net: J3.2 (Pin_2), R7.2
- new net: J2.1 (Pin_1), R6.2
- new net: J1.2 (Pin_2), R4.2
- new net: J1.1 (Pin_1), R5.2
- new net: J2.2 (Pin_2), R7.2
Other:
- moved on the sheet: C5, C8, D1, R44, U11
